File: pcb/HEXTIr_v1.sch (EAGLE design)
At the start: 27 parts, among them CN1 HEX-BUS, IC1 ATMEGA328

Commit message: PCB and schematic updates
Parts:
- CN1: device ti994a:HEX-BUS -> ti_cc40:HEX-BUS
- R2, R3, R4: value (none) -> 1800
- R5, R6, R7: value (none) -> 3300
Connections:
- removed net N$14: C5.2
- removed net N$15: C6.2
- removed net N$16: C7.2
- net GND: now also C5.2, C6.2, C7.2, CN1.GND
- net N$13: now also CN1.BAV; no longer CN1.!BAV
Other:
- note added: "HEX-TI-r SD The Texas Instruments HEX-BUS SD Drive"
- note removed: "PS2 to Parallel/Serial Keyboard Encoder"
- moved on the sheet: R5, R6, R7
