File: pcb/HEXTIr_v1.sch (EAGLE design)
At the start: 27 parts, among them CN1 HEX-BUS, IC1 ATMEGA328

Commit message: PCB tweaks
Parts:
- added GOLD_ORB_SM1: Open Source Hardware, oshw:OSHWLOGOLOGO5MM
Changed lines of the file:
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@@
 <layer number="121" name="_tsilk" color="7" fill="1" visible="yes" active="yes"/>
 <layer number="122" name="_bsilk" color="7" fill="1" visible="yes" active="yes"/>
+<layer number="125" name="_tNames" color="7" fill="1" visible="yes" active="yes"/>
+<layer number="144" name="Drill_legend" color="7" fill="1" visible="yes" active="yes"/>
 <layer number="151" name="HeatSink" color="7" fill="1" visible="yes" active="yes"/>
 <layer number="200" name="200bmp" color="7" fill="1" visible="yes" active="yes"/>
@@
 <layer number="207" name="207bmp" color="8" fill="10" visible="yes" active="yes"/>
 <layer number="208" name="208bmp" color="9" fill="10" visible="yes" active="yes"/>
+<layer number="209" name="209bmp" color="7" fill="1" visible="yes" active="yes"/>
+<layer number="210" name="210bmp" color="7" fill="1" visible="yes" active="yes"/>
+<layer number="211" name="211bmp" color="7" fill="1" visible="yes" active="yes"/>
+<layer number="212" name="212bmp" color="7" fill="1" visible="yes" active="yes"/>
+<layer number="213" name="213bmp" color="7" fill="1" visible="yes" active="yes"/>
+<layer number="214" name="214bmp" color="7" fill="1" visible="yes" active="yes"/>
+<layer number="215" name="215bmp" color="7" fill="1" visible="yes" active="yes"/>
 <layer number="216" name="SMD16" color="7" fill="1" visible="yes" active="yes"/>
 <layer number="250" name="Descript" color="3" fill="1" visible="no" active="no"/>
@@
 <part name="GND13" library="supply1" deviceset="GND" device=""/>
 <part name="CN1" library="ti_cc40" deviceset="HEX-BUS" device=""/>
+<part name="GOLD_ORB_SM1" library="oshw" deviceset="OSHWLOGO" device="LOGO5MM" value="Open Source Hardware"/>
 </parts>
 <sheets>
@@
 <instance part="GND13" gate="1" x="160.02" y="5.08"/>
 <instance part="CN1" gate="G$1" x="132.08" y="170.18"/>
+<instance part="GOLD_ORB_SM1" gate="G$1" x="226.06" y="48.26"/>
 </instances>
 <busses>
