File: pcb/HEXTIr_v1.sch (EAGLE design)
At the start: 28 parts, among them CN1 HEX-BUS, IC1 ATMEGA328

Commit message: Working Arduino codebase
Connections:
- net N$10 renamed D2
- net N$11 renamed D3
- net N$12 renamed !HSK
- net N$13 renamed BAV
- net N$8 renamed D0
- net N$9 renamed D1
Changed lines of the file:
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@@
 </segment>
 </net>
-<net name="N$8" class="0">
+<net name="D0" class="0">
 <segment>
 <pinref part="IC1" gate="G$1" pin="PC0(ADC0)"/>
@@
 </segment>
 </net>
-<net name="N$9" class="0">
+<net name="D1" class="0">
 <segment>
 <pinref part="IC1" gate="G$1" pin="PC1(ADC1)"/>
@@
 </segment>
 </net>
-<net name="N$10" class="0">
+<net name="D2" class="0">
 <segment>
 <pinref part="IC1" gate="G$1" pin="PC2(ADC2)"/>
@@
 </segment>
 </net>
-<net name="N$11" class="0">
+<net name="D3" class="0">
 <segment>
 <pinref part="IC1" gate="G$1" pin="PC3(ADC3)"/>
@@
 </segment>
 </net>
-<net name="N$12" class="0">
+<net name="!HSK" class="0">
 <segment>
 <wire x1="121.92" y1="177.8" x2="106.68" y2="177.8" width="0.1524" layer="91"/>
@@
 </segment>
 </net>
-<net name="N$13" class="0">
+<net name="BAV" class="0">
 <segment>
 <pinref part="IC1" gate="G$1" pin="PC5(ADC5/SCL)"/>
