File: pcb/HEXTIr_v1.brd (EAGLE design)
At the start: 71.1 x 38.1 mm, 27 parts, among them CN1 HEX-BUS, IC1 ATMEGA328

Commit message: PCB and schematic updates
Parts:
- CN1: device ti994a:HEX-BUS -> ti_cc40:HEX-BUS
- R2, R3, R4: value (none) -> 1800
- R5, R6, R7: value (none) -> 3300
Connections:
- removed net N$14: C5.2
- removed net N$15: C6.2
- removed net N$16: C7.2
- net GND: now also C5.2, C6.2, C7.2, CN1.4

Commit message: PCB tweaks
Parts:
- added GOLD_ORB_SM1: Open Source Hardware, oshw:OSHW_5MM
Changed lines of the file:
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@@
 <layer number="121" name="_tsilk" color="7" fill="1" visible="yes" active="yes"/>
 <layer number="122" name="_bsilk" color="7" fill="1" visible="yes" active="yes"/>
+<layer number="125" name="_tNames" color="7" fill="1" visible="yes" active="yes"/>
+<layer number="144" name="Drill_legend" color="7" fill="1" visible="yes" active="yes"/>
 <layer number="151" name="HeatSink" color="7" fill="1" visible="yes" active="yes"/>
 <layer number="200" name="200bmp" color="7" fill="1" visible="yes" active="yes"/>
@@
 <layer number="207" name="207bmp" color="8" fill="10" visible="yes" active="yes"/>
 <layer number="208" name="208bmp" color="9" fill="10" visible="yes" active="yes"/>
+<layer number="209" name="209bmp" color="7" fill="1" visible="yes" active="yes"/>
+<layer number="210" name="210bmp" color="7" fill="1" visible="yes" active="yes"/>
+<layer number="211" name="211bmp" color="7" fill="1" visible="yes" active="yes"/>
+<layer number="212" name="212bmp" color="7" fill="1" visible="yes" active="yes"/>
+<layer number="213" name="213bmp" color="7" fill="1" visible="yes" active="yes"/>
+<layer number="214" name="214bmp" color="7" fill="1" visible="yes" active="yes"/>
+<layer number="215" name="215bmp" color="7" fill="1" visible="yes" active="yes"/>
 <layer number="216" name="SMD16" color="7" fill="1" visible="yes" active="yes"/>
 <layer number="250" name="Descript" color="3" fill="1" visible="no" active="no"/>
@@
 <attribute name="VALUE" x="-29.845" y="-41.91" size="1.27" layer="27" ratio="10" rot="R270"/>
 </element>
+<element name="GOLD_ORB_SM1" library="oshw" package="OSHW_5MM" value="Open Source Hardware" x="-29.21" y="-56.515" smashed="yes">
+<attribute name="VALUE" x="-29.21" y="-53.975" size="0.6096" layer="27" align="bottom-center"/>
+</element>
 </elements>

Commit message: Working Arduino codebase
Connections:
- net N$10 renamed D2
- net N$11 renamed D3
- net N$12 renamed !HSK
- net N$13 renamed BAV
- net N$8 renamed D0
- net N$9 renamed D1
Changed lines of the file:
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@@
 <wire x1="8.9662" y1="-39.9542" x2="8.382" y2="-39.37" width="0.4064" layer="16"/>
 </signal>
-<signal name="N$8">
+<signal name="D0">
 <contactref element="IC1" pad="23"/>
 <wire x1="-31.75" y1="-50.8" x2="-27.94" y2="-54.61" width="0.254" layer="1"/>
@@
 <contactref element="CN1" pad="1"/>
 </signal>
-<signal name="N$9">
+<signal name="D1">
 <contactref element="IC1" pad="24"/>
 <wire x1="-31.75" y1="-48.26" x2="-19.05" y2="-48.26" width="0.254" layer="16"/>
@@
 <contactref element="CN1" pad="2"/>
 </signal>
-<signal name="N$10">
+<signal name="D2">
 <contactref element="IC1" pad="25"/>
 <wire x1="-34.29" y1="-45.72" x2="-33.02" y2="-46.99" width="0.254" layer="16"/>
@@
 <contactref element="CN1" pad="7"/>
 </signal>
-<signal name="N$11">
+<signal name="D3">
 <contactref element="IC1" pad="26"/>
 <wire x1="-34.29" y1="-43.18" x2="-33.02" y2="-44.45" width="0.254" layer="16"/>
@@
 <contactref element="CN1" pad="8"/>
 </signal>
-<signal name="N$12">
+<signal name="!HSK">
 <contactref element="IC1" pad="27"/>
 <wire x1="-34.29" y1="-50.8" x2="-33.02" y2="-49.53" width="0.254" layer="1"/>
@@
 <contactref element="CN1" pad="5"/>
 </signal>
-<signal name="N$13">
+<signal name="BAV">
 <contactref element="IC1" pad="28"/>
 <wire x1="-31.75" y1="-45.72" x2="-30.48" y2="-44.45" width="0.254" layer="1"/>
